File: kicad/nfc.kicad_sch (KiCad schematic)
At the start: 3 parts, among them U1 NT3H2111W0FHKH

Commit message: sept 26
Parts:
- added Cap1: 150-220nf, Capacitor_SMD:C_0201_0603Metric, symbol Device:C_Small
- added L1: L_Small, antenna:ftprnt, symbol Device:L_Small
- added R1, R2, R3: 5k ohm, Resistor_SMD:R_0201_0603Metric, symbol Device:R
- Con1: renamed from Con; footprint (none) -> Connector_Hirose:Hirose_DF13-05P-1.25DSA_1x05_P1.25mm_Vertical
Connections:
- net vout is gone; now on net +2V8: D1.1 (K), U1.7 (VOUT)
- net FD: now also R3.2
- net GND: now also Cap1.2
- net SCL: now also R1.2
- net SDA: now also R2.2
- net LA: now reaches U1.1 (LA)
- net LA: now also L1.1
- net LB: now reaches U1.8 (LB)
- net LB: now also L1.2
- net +3.3V renamed +2V8
- net +2V8: now also Cap1.1, R1.1, R2.1, R3.1
Other:
- note added: "Custom foot print for antenna"
- note added: "Traces for later i2c communication"
- moved on the sheet: D1, U1

Commit message: done
Parts:
- Cap1: value 150-220nf -> 180 nf
Changed lines of the file:
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@@
 			)
 		)
-		(property "Value" "150-220nf"
+		(property "Value" "180 nf"
 			(at 100.076 54.61 0)
 			(show_name no)

Commit message: ok kinda done gonna tune right now again
Parts:
- Cap1: footprint Capacitor_SMD:C_0201_0603Metric -> Capacitor_SMD:C_0603_1608Metric
- Con1: value trace -> Conn_01x05_Pin
- L1: footprint antenna:ftprnt -> footprint:ftprnt
- R1, R2, R3: footprint Resistor_SMD:R_0201_0603Metric -> Resistor_SMD:R_0603_1608Metric
Changed lines of the file:
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@@
 			)
 		)
-		(property "Footprint" "antenna:ftprnt"
+		(property "Footprint" "footprint:ftprnt"
 			(at 106.68 81.28 0)
 			(hide yes)
@@
 			)
 		)
-		(property "Value" "trace"
+		(property "Value" "Conn_01x05_Pin"
 			(at 186.944 54.356 0)
 			(show_name no)
@@
 			)
 		)
-		(property "Footprint" "Resistor_SMD:R_0201_0603Metric"
+		(property "Footprint" "Resistor_SMD:R_0603_1608Metric"
 			(at 239.522 71.12 90)
 			(hide yes)
@@
 			)
 		)
-		(property "Footprint" "Resistor_SMD:R_0201_0603Metric"
+		(property "Footprint" "Resistor_SMD:R_0603_1608Metric"
 			(at 228.092 71.12 90)
 			(hide yes)
@@
 			)
 		)
-		(property "Footprint" "Resistor_SMD:R_0201_0603Metric"
+		(property "Footprint" "Resistor_SMD:R_0603_1608Metric"
 			(at 250.952 71.12 90)
 			(hide yes)
@@
 			)
 		)
-		(property "Footprint" "Capacitor_SMD:C_0201_0603Metric"
+		(property "Footprint" "Capacitor_SMD:C_0603_1608Metric"
 			(at 104.14 62.23 0)
 			(hide yes)
